File: IntegratedCavityPID.kicad_pcb (KiCad board)
At the start: 4 copper layers, 152.5 x 152.5 mm, 452 parts, among them IC1 AD835ARZ, IC10 PE4250MLI-Z, IC11 PE4250MLI-Z, IC12 PE4250MLI-Z, IC13 PE4250MLI-Z, IC15 LT3090EMSE#PBF, IC16 LT3085EMS8E#TRPBF, IC2 LT3085EMS8E#TRPBF, IC5 THS4521IDR, IC6 ADS8863IDGS, IC7 THS4521IDR, IC8 ADS8863IDGS, IC9 LTC6655BHMS8-4.096#PBF, J1 U254-051T-4BH83-S1S, J10 Conn_01x12_Male, J11 SMA, J12 SMA, J13 RFShield_OnePiece, J14 RFShield_OnePiece, J15 u.fl, J16 Conn_Coaxial, J17 SMA, J18 u.fl, J19 u.fl, J2 U254-051T-4BH83-S1S, J20 B-2100N06P-B111, J21 B-2100N06P-B111, J22 mux, J23 Conn_Coaxial, J24 Conn_Coaxial, J25 Conn_01x04, J26 AudioJack3, J27 Conn_Coaxial, J28 Conn_Coaxial, J29 Conn_01x04, J3 Conn_Coaxial, J30 Conn_01x06, J4 Conn_Coaxial, J5 debug, J6 Clock_in, J7 Conn_01x08, J8 Conn_01x30_Male, J9 Conn_01x21_Male, Q1 MMBT3906, Q2 mmbt3904, Q3 2SCR573, Q4 2SAR573, Q5 MMBT3906, Q6 mmbt3904, Q7 2SCR573, Q8 2SAR573, T1 MABA-007532-CF18A0, T2 MABA-007532-CF18A0, U1 CH32V307RCT6, U10 ADA4841-2, U11 OPA388, U12 ADR421ARZ, U13 THS4281, U14 PHA-13LN, U15 PAT1220-C-6DB, U16 PAT1220-C-6DB, U17 PAT1220-C-8DB, U18 74HC04, U19 PAT1220-C-8DB, U2 PHA-13LN, U20 PAT1220-C-8DB, U21 MAX5719xSD, U22 OPA388, U23 THS4551xRGT, U24 THS4551xRGT, U25 LT3080xDD, U3 PHA-13LN, U4 74HC4051M/TR, U5 ADA4075-2, U6 ADG419BR, U7 ADA4075-2, U8 MAX5719xSD, U9 74HC04, Y1 X32258MOB4SI

Commit message: Preliminary layout of analog portions
Parts:
- removed IC16, IC2: LT3085EMS8E#TRPBF, SamacSys_Parts:SOP65P490X110-9N
- added D16: SS210, Diode_SMD:D_SMA, F.Cu at (-207.5, 101.2)
- added J31: Conn_01x02, Connector_PinHeader_2.54mm:PinHeader_1x02_P2.54mm_Vertical, F.Cu at (-202.8, 105.0)
- added J32: SMA, Connector_Coaxial:SMA_Amphenol_132134-10_Vertical, F.Cu at (-162.0, 92.5)
- added L12: SWPA6028S180MT, Inductor_SMD:L_Bourns-SRN6028, F.Cu at (-199.8, 94.0)
- added R165: 0805W8F1004T5E, Resistor_SMD:R_0805_2012Metric, F.Cu at (-198.8, 67.2)
- added U26: LT3080xDD, Package_DFN_QFN:DFN-8-1EP_3x3mm_P0.5mm_EP1.66x2.38mm, F.Cu at (-90.5, 4.72)
- C45: footprint Capacitor_SMD:C_1206_3216Metric -> Capacitor_SMD:C_1210_3225Metric_Pad1.33x2.70mm_HandSolder
- J26: value AudioJack3 -> SJ1-3514-SMT-TR; footprint Connector_Audio:Jack_3.5mm_CUI_SJ-3524-SMT_Horizontal -> SamacSys_Parts:SJ13514SMTTR
- R11: value 470k -> 0805W8F2204T5E
- R12: value 33k -> 0
- R145: value 33k -> 56k
- moved U24 120.4 mm to (-245.2, 43.5)
- moved U23 116.5 mm to (-243.8, 43.7)
- moved R147 92.9 mm to (-103.5, -10.3), turned to -90 degrees
- moved C101 89.9 mm to (-84.0, 6.22), turned to -90 degrees
- moved C151 86.9 mm to (-96.6, 2.23), turned to 90 degrees
- moved J28 85.8 mm to (-107.5, -7.53), turned to 180 degrees
- moved C155 82.3 mm to (-100.5, 5.47), turned to 180 degrees
- moved J27 82.0 mm to (-107.3, 2.98), turned to 180 degrees
- moved C152 81.7 mm to (-97.0, -10.1), turned to 90 degrees
- moved C82 79.6 mm to (-73.5, -0.28), turned to 90 degrees
- moved C49 79.1 mm to (-71.0, -4.78), turned to -90 degrees
- moved C132 79.1 mm to (-86.5, 1.23), turned to 90 degrees
- moved R146 76.7 mm to (-101.5, -10.3), turned to 90 degrees
- moved C120 75.0 mm to (-84.5, -10.8), turned to -90 degrees
- moved C51 74.0 mm to (-73.5, -4.28), turned to -90 degrees
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Connections:
- C101 pad 2: Net-(C101-Pad2) -> GND
- C120 pad 2: Net-(C120-Pad2) -> Net-(IC15-Pad1)
- C131 pad 1: Net-(C120-Pad2) -> Net-(IC15-Pad1)
- C132 pad 2: Net-(C101-Pad2) -> GND
- C133 pad 1: Net-(C120-Pad2) -> Net-(IC15-Pad1)
- C134 pad 2: Net-(C101-Pad2) -> GND
- C135 pad 2: Net-(C101-Pad2) -> GND
- C136 pad 1: Net-(C120-Pad2) -> Net-(IC15-Pad1)
- C137 pad 2: Net-(C137-Pad2) -> GND
- C147 pad 1: Net-(R138-Pad2) -> /main/AnalogLoop/Piezo_Drive/piezo_slow
- C158 pad 1: Net-(R138-Pad2) -> /main/AnalogLoop/Piezo_Drive/piezo_slow
- C40 pad 2: Net-(C137-Pad2) -> Net-(C40-Pad2)
- C41 pad 2: Net-(C137-Pad2) -> Net-(C40-Pad2)
- C42 pad 2: Net-(C137-Pad2) -> GND
- C43 pad 2: Net-(C137-Pad2) -> GND
- C44 pad 2: Net-(C137-Pad2) -> GND
- C50 pad 2: Net-(C101-Pad2) -> GND
- C67 pad 1: /main/AnalogLoop/Piezo_Drive/bias_l -> Net-(C67-Pad1)
- C82 pad 2: Net-(C101-Pad2) -> GND
- D7 pad 2: /main/AnalogLoop/Piezo_Drive/bias_l -> Net-(C67-Pad1)
- L2 pad 2: Net-(C120-Pad2) -> Net-(IC15-Pad1)
- R12 pad 1: Net-(R11-Pad2) -> Net-(R12-Pad1)
- R138 pad 2: Net-(R138-Pad2) -> /main/AnalogLoop/Piezo_Drive/piezo_slow
- R162 pad 2: unconnected-(R162-Pad2) -> /main/AnalogLoop/Piezo_Drive/piezo_fast
- R92 pad 2: /main/AnalogLoop/Piezo_Drive/bias_l -> Net-(C67-Pad1)
- U25 pad 1: unconnected-(U25-Pad1) -> +28V
- U25 pad 2: unconnected-(U25-Pad2) -> +28V
- U25 pad 3: unconnected-(U25-Pad3) -> +28V
- U25 pad 4: unconnected-(U25-Pad4) -> Net-(C45-Pad1)
- U25 pad 5: unconnected-(U25-Pad5) -> Net-(C137-Pad1)
- U25 pad 7: unconnected-(U25-Pad7) -> Net-(C137-Pad1)
- U25 pad 8: unconnected-(U25-Pad8) -> Net-(C137-Pad1)
- U25 pad 9: unconnected-(U25-Pad9) -> +28V
Routing:
- net +28V: track 0.00 -> 68.8 mm
- net -5VA: track 11.2 -> 49.1 mm
- net Net-(IC15-Pad1): track 0.00 -> 35.6 mm, vias 0 -> 2
- net +5VA: track 44.0 -> 72.6 mm
- net /main/AnalogLoop/Piezo_Drive/piezo_slow: track 0.00 -> 22.3 mm
- net Net-(C101-Pad1): track 0.00 -> 20.7 mm
- net Ref_Buf: track 3.63 -> 19.8 mm
- net /main/AnalogLoop/Piezo_Drive/piezo_fast: track 0.00 -> 14.1 mm
- net Net-(R105-Pad2): track 0.00 -> 13.9 mm
- net Net-(C20-Pad2): track 0.00 -> 11.8 mm
- net Net-(C68-Pad2): track 0.00 -> 11.4 mm
- net /main/AnalogLoop/Piezo_Drive/bias_h: track 0.00 -> 10.4 mm
- net Net-(C50-Pad1): track 0.00 -> 10.2 mm
- net Net-(C107-Pad1): track 0.00 -> 10.2 mm
- net Net-(C49-Pad1): track 0.00 -> 10.1 mm
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