File: AnalogLoop.kicad_sch (KiCad schematic)
At the start: 24 parts, among them J18 u.fl, J19 u.fl, U5 ADA4075-2, U6 ADG419BR

Commit message: Analog section complete!
Parts:
- removed C25: 0.1uF, Capacitor_SMD:C_0603_1608Metric_Pad1.08x0.95mm_HandSolder, symbol Device:C
- removed U6: ADG419BR, Package_SO:SOIC-8_3.9x4.9mm_P1.27mm, symbol Analog_Switch:ADG419BR
- added J?: Conn_01x03, Connector_PinHeader_2.54mm:PinHeader_1x03_P2.54mm_Vertical, symbol Connector_Generic:Conn_01x03
- added R167, R168: dnp, Resistor_SMD:R_0805_2012Metric, symbol Device:R
- added R97: 0, Resistor_SMD:R_0805_2012Metric, symbol Device:R
- added TP6: tp, TestPoint:TestPoint_Pad_D1.0mm, symbol Connector:TestPoint
- added U6: ADG1419BRM, Package_SO:MSOP-8_3x3mm_P0.65mm, symbol Analog_Switch:ADG419BRM
Connections:
- net +5VA: now also U6.4 (V+)
- net -5VA: now also U6.7 (V-)
- net DAC1_output: now also R167.2
- net GND: now also J?.1 (Pin_1), J?.3 (Pin_3), U6.3 (GND)
- net at R87.2: now also U6.1
- net at R152.1: now also U6.2
- net at C74.2, J19.1 (In), R86.2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: now also U6.8
- net Piezo_Drive/input renamed Piezo_Drive/fast_in_B
- net Piezo_Drive/offset renamed Piezo_Drive/slow_in
- net Piezo_Drive/slow_in: now also R168.1
- new net: J?.2 (Pin_2), U6.6
- new net: TP6.1, U6.5 (VL)
- new net DAC2_output: R168.2, R97.2
- new net Piezo_Drive/fast_in_A: R167.1, R97.1
Other:
- sheet Piezo_Drive ports: added fast_in_A, fast_in_B, slow_in; removed input, offset
- note added: "For ADG1419 pin5 is NC No VL needed"
- moved on the sheet: C26, C27, R152, R153

Commit message: Digital section half finished
Parts:
- gave numbers to parts that had none: 1
Changed lines of the file:
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@@
   (symbol (lib_id "Connector_Generic:Conn_01x03") (at 147.32 33.02 90) (unit 1)
     (in_bom yes) (on_board yes) (fields_autoplaced)
-    (property "Reference" "J?" (id 0) (at 152.4 31.7499 90)
+    (property "Reference" "J34" (id 0) (at 152.4 31.7499 90)
       (effects (font (size 1.27 1.27)) (justify right))
     )

Commit message: Version 1.0 submitted to JLCPCB
Parts:
- J18, J19: value u.fl -> DNP U.FL
- R148, R151, R152, R153, R84, R87, R97: value 0 -> 0R
Changed lines of the file:
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@@
       (effects (font (size 1.27 1.27)) (justify right))
     )
-    (property "Value" "0" (id 1) (at 196.85 43.1799 0)
+    (property "Value" "0R" (id 1) (at 196.85 43.1799 0)
       (effects (font (size 1.27 1.27)) (justify right))
     )
@@
       (effects (font (size 1.27 1.27)) (justify left))
     )
-    (property "Value" "u.fl" (id 1) (at 69.85 105.41 0)
+    (property "Value" "DNP U.FL" (id 1) (at 69.85 105.41 0)
       (effects (font (size 1.27 1.27)) (justify left))
     )
@@
     (in_bom yes) (on_board yes) (fields_autoplaced)
     (property "Reference" "R87" (id 0) (at 161.29 49.53 90))
-    (property "Value" "0" (id 1) (at 161.29 52.07 90))
+    (property "Value" "0R" (id 1) (at 161.29 52.07 90))
     (property "Footprint" "Resistor_SMD:R_0805_2012Metric" (id 2) (at 161.29 54.102 90)
       (effects (font (size 1.27 1.27)) hide)
@@
       (effects (font (size 1.27 1.27)) (justify left))
     )
-    (property "Value" "u.fl" (id 1) (at 125.73 46.99 0)
+    (property "Value" "DNP U.FL" (id 1) (at 125.73 46.99 0)
       (effects (font (size 1.27 1.27)) (justify left))
     )
@@
     (in_bom yes) (on_board yes) (fields_autoplaced)
     (property "Reference" "R151" (id 0) (at 40.64 44.45 90))
-    (property "Value" "0" (id 1) (at 40.64 46.99 90))
+    (property "Value" "0R" (id 1) (at 40.64 46.99 90))
     (property "Footprint" "Resistor_SMD:R_0805_2012Metric" (id 2) (at 40.64 52.578 90)
       (effects (font (size 1.27 1.27)) hide)
@@
     (in_bom yes) (on_board yes)
     (property "Reference" "R97" (id 0) (at 180.34 72.39 90))
-    (property "Value" "0" (id 1) (at 182.88 72.39 90))
+    (property "Value" "0R" (id 1) (at 182.88 72.39 90))
     (property "Footprint" "Resistor_SMD:R_0805_2012Metric" (id 2) (at 181.102 72.39 90)
       (effects (font (size 1.27 1.27)) hide)
@@
       (effects (font (size 1.27 1.27)) (justify left))
     )
-    (property "Value" "0" (id 1) (at 134.62 66.0399 0)
+    (property "Value" "0R" (id 1) (at 134.62 66.0399 0)
       (effects (font (size 1.27 1.27)) (justify left))
     )
@@
       (effects (font (size 1.27 1.27)) (justify right))
     )
-    (property "Value" "0" (id 1) (at 35.56 76.1999 0)
+    (property "Value" "0R" (id 1) (at 35.56 76.1999 0)
       (effects (font (size 1.27 1.27)) (justify right))
     )
@@
     (in_bom yes) (on_board yes) (fields_autoplaced)
     (property "Reference" "R84" (id 0) (at 80.01 44.45 90))
-    (property "Value" "0" (id 1) (at 80.01 46.99 90))
+    (property "Value" "0R" (id 1) (at 80.01 46.99 90))
     (property "Footprint" "Resistor_SMD:R_0805_2012Metric" (id 2) (at 80.01 52.578 90)
       (effects (font (size 1.27 1.27)) hide)
