File: DataConverters.kicad_sch (KiCad schematic)
At the start: 7 parts, among them J20 B-2100N06P-B111, J21 B-2100N06P-B111, U9 74HC04

Commit message: Analog section complete!
Parts:
- added JP15: sjp, Jumper:SolderJumper-2_P1.3mm_Open_RoundedPad1.0x1.5mm, symbol Jumper:SolderJumper_2_Open
Connections:
- net ADC_buffered_2/In_pos: now also JP15.2 (B)
- net Error_Buffered: now also JP15.1 (A)
Changed lines of the file:
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@@
+    (stroke (width 0) (type default) (color 0 0 0 0))
+  )
+  (wire (pts (xy 93.98 92.71) (xy 97.79 92.71))
     (stroke (width 0) (type default) (color 0 0 0 0))
   )
@@
     )
   )
+  (global_label "Error_Buffered" (shape input) (at 93.98 92.71 180) (fields_autoplaced)
+    (effects (font (size 1.27 1.27)) (justify right))
+    (property "Intersheet References" "${INTERSHEET_REFS}" (id 0) (at 77.9598 92.7894 0)
+      (effects (font (size 1.27 1.27)) (justify right) hide)
+    )
+  )
   (global_label "ADC1_DOUT" (shape input) (at 135.89 43.18 0) (fields_autoplaced)
     (effects (font (size 1.27 1.27)) (justify left))
@@
     )
   )
+  (symbol (lib_id "Jumper:SolderJumper_2_Open") (at 101.6 92.71 0) (unit 1)
+    (in_bom yes) (on_board yes)
+    (property "Reference" "JP15" (id 0) (at 101.6 87.63 0))
+    (property "Value" "sjp" (id 1) (at 101.6 90.17 0))
+    (property "Footprint" "Jumper:SolderJumper-2_P1.3mm_Open_RoundedPad1.0x1.5mm" (id 2) (at 101.6 92.71 0)
+      (effects (font (size 1.27 1.27)) hide)
+    )
+    (property "Datasheet" "~" (id 3) (at 101.6 92.71 0)
+      (effects (font (size 1.27 1.27)) hide)
+    )
+    (pin "1")
+    (pin "2")
+  )
   (symbol (lib_id "Device:C") (at 259.08 133.35 0) (mirror x) (unit 1)

Commit message: Digital section half finished
Parts:
- added JP16: sjp, Jumper:SolderJumper-2_P1.3mm_Open_RoundedPad1.0x1.5mm, symbol Jumper:SolderJumper_2_Open
Connections:
- net Error_Buffered: now also JP16.1 (A); no longer JP15.1 (A)
- new net: JP15.1 (A), JP16.2 (B)
Changed lines of the file:
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@@
   (junction (at 270.51 119.38) (diameter 0) (color 0 0 0 0)
   )
+  (wire (pts (xy 93.98 92.71) (xy 97.79 92.71))
+    (stroke (width 0) (type default) (color 0 0 0 0))
+  )
   (wire (pts (xy 128.27 139.7) (xy 130.81 139.7))
     (stroke (width 0) (type default) (color 0 0 0 0))
   )
-  (wire (pts (xy 93.98 92.71) (xy 97.79 92.71))
+  (wire (pts (xy 78.74 92.71) (xy 86.36 92.71))
     (stroke (width 0) (type default) (color 0 0 0 0))
   )
@@
     )
   )
-  (global_label "Error_Buffered" (shape input) (at 93.98 92.71 180) (fields_autoplaced)
-    (effects (font (size 1.27 1.27)) (justify right))
-    (property "Intersheet References" "${INTERSHEET_REFS}" (id 0) (at 77.9598 92.7894 0)
+  (global_label "Error_Buffered" (shape input) (at 78.74 92.71 180) (fields_autoplaced)
+    (effects (font (size 1.27 1.27)) (justify right))
+    (property "Intersheet References" "${INTERSHEET_REFS}" (id 0) (at 62.7198 92.7894 0)
       (effects (font (size 1.27 1.27)) (justify right) hide)
     )
@@
     (pin "7")
   )
+  (symbol (lib_id "Jumper:SolderJumper_2_Open") (at 90.17 92.71 0) (unit 1)
+    (in_bom yes) (on_board yes)
+    (property "Reference" "JP16" (id 0) (at 90.17 87.63 0))
+    (property "Value" "sjp" (id 1) (at 90.17 90.17 0))
+    (property "Footprint" "Jumper:SolderJumper-2_P1.3mm_Open_RoundedPad1.0x1.5mm" (id 2) (at 90.17 92.71 0)
+      (effects (font (size 1.27 1.27)) hide)
+    )
+    (property "Datasheet" "~" (id 3) (at 90.17 92.71 0)
+      (effects (font (size 1.27 1.27)) hide)
+    )
+    (pin "1")
+    (pin "2")
+  )
   (symbol (lib_id "74xx:74HC04") (at 227.33 105.41 0) (unit 1)

Commit message: First finished draft
Parts:
- added J41: Conn_02x03_Odd_Even, Connector_PinHeader_2.00mm:PinHeader_2x03_P2.00mm_Vertical, symbol Connector_Generic:Conn_02x03_Odd_Even
- added JP20: sjp, Jumper:SolderJumper-2_P1.3mm_Open_RoundedPad1.0x1.5mm, symbol Jumper:SolderJumper_2_Open
- added R180: dnp, Resistor_SMD:R_0805_2012Metric, symbol Device:R
- added TP11, TP14, TP7, TP9: tp, TestPoint:TestPoint_Pad_D1.0mm, symbol Connector:TestPoint
Connections:
- net ADC_buffered_2/In_pos: now also R180.2; no longer JP15.2 (B)
- net DAC2_SCLK: now also U9.3; no longer U9.5
- net GND: now also J41.1 (Pin_1), J41.2 (Pin_2)
- net at JP16.2 (B): now also JP20.1 (A); no longer JP15.1 (A)
- net at U9.6: now also TP9.1; no longer R155.1
- net at U9.10: now also J41.4 (Pin_4)
- net at U9.11: now also J41.6 (Pin_6)
- net at U9.12: now also J41.5 (Pin_5)
- net at U9.13: now also J41.3 (Pin_3)
- net at U9.4: now also R155.1
- net at U9.1: now also TP11.1
- net at U9.2: now also TP14.1
- new net: JP15.2 (B), JP20.2 (B), R180.1
- new net: TP7.1, U9.5
- new net reflection_DC: JP15.1 (A)
Other:
- moved on the sheet: J20, J21, JP16, R154, R155, U9A, U9B, U9C, U9D, U9E, U9F
