File: MAX8863_core.kicad_sch (KiCad schematic)
At the start: 25 parts, among them IC5 THS4521IDR, IC6 ADS8863IDGS, J3 Conn_Coaxial, U23 THS4551xRGT

Commit message: Analog section complete!
Parts:
- removed IC5: THS4521IDR, SamacSys_Parts:SOIC127P600X175-8N, symbol SamacSys_Parts:THS4521IDR
Connections:
- net +5VA: now also U23.5 (VS+), U23.6 (VS+), U23.7 (VS+), U23.8 (VS+)
- net GND: now also U23.13 (VS-), U23.14 (VS-), U23.15 (VS-), U23.16 (VS-), U23.17 (EP)
- net PDn: now also U23.9 (VOCM)
- net Vcom: now also U23.12 (~{PD})
- net at C78.2, R112.1: now also U23.1 (FB-); no longer R114.2
- net at C79.1, R111.1: now also U23.3 (IN-)
- net at C79.2, R113.1: now also U23.4 (FB+); no longer R115.2
- net at U23.10 (OUT+): now also R115.2
- net at U23.11 (OUT-): now also R114.2
- net at U23.2 (IN+): now also C78.1, R110.1
Other:
- moved on the sheet: C75, C78, C79, J3, R107, R108, R109, R110, R111, R112, R113, TP3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

Commit message: Version 1.0 submitted to JLCPCB
Parts:
- C78, C79: value 1nF C0G -> CGA4C2C0G1H102JT0Y0N
- C81: value 10nF C0G -> CGA4C2C0G1H103JT0Y0N
- J3: value Conn_Coaxial -> DNP SMA
- R107: value 0 -> 0R
- U23: value THS4551xRGT -> THS4551IRGTR
Changed lines of the file:
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@@
       (effects (font (size 1.27 1.27)) (justify left))
     )
-    (property "Value" "1nF C0G" (id 1) (at 85.09 138.43 90)
+    (property "Value" "CGA4C2C0G1H102JT0Y0N" (id 1) (at 85.09 138.43 90)
       (effects (font (size 1.27 1.27)) (justify left))
     )
@@
       (effects (font (size 1.27 1.27)) (justify left))
     )
-    (property "Value" "THS4551xRGT" (id 1) (at 97.79 116.84 0)
+    (property "Value" "THS4551IRGTR" (id 1) (at 97.79 116.84 0)
       (effects (font (size 1.27 1.27)) (justify left))
     )
@@
       (effects (font (size 1.27 1.27)) (justify left))
     )
-    (property "Value" "THS4551xRGT" (id 1) (at 208.28 124.4599 0)
+    (property "Value" "THS4551IRGTR" (id 1) (at 208.28 124.4599 0)
       (effects (font (size 1.27 1.27)) (justify left))
     )
@@
     (in_bom yes) (on_board yes) (fields_autoplaced)
     (property "Reference" "R107" (id 0) (at 34.29 83.82 90))
-    (property "Value" "0" (id 1) (at 34.29 86.36 90))
+    (property "Value" "0R" (id 1) (at 34.29 86.36 90))
     (property "Footprint" "Resistor_SMD:R_0805_2012Metric" (id 2) (at 34.29 88.392 90)
       (effects (font (size 1.27 1.27)) hide)
@@
       (effects (font (size 1.27 1.27)) (justify left))
     )
-    (property "Value" "1nF C0G" (id 1) (at 82.55 78.74 90)
+    (property "Value" "CGA4C2C0G1H102JT0Y0N" (id 1) (at 82.55 78.74 90)
       (effects (font (size 1.27 1.27)) (justify left))
     )
@@
     (in_bom yes) (on_board yes) (fields_autoplaced)
     (property "Reference" "J3" (id 0) (at 42.2274 133.35 0))
-    (property "Value" "Conn_Coaxial" (id 1) (at 42.2274 130.81 0))
+    (property "Value" "DNP SMA" (id 1) (at 42.2274 130.81 0))
     (property "Footprint" "Connector_Coaxial:SMA_Amphenol_132134_Vertical" (id 2) (at 41.91 125.73 0)
       (effects (font (size 1.27 1.27)) hide)
@@
       (effects (font (size 1.27 1.27)) (justify left))
     )
-    (property "Value" "10nF C0G" (id 1) (at 135.89 120.65 90)
-      (effects (font (size 1.27 1.27)) (justify left))
-    )
+    (property "Value" "CGA4C2C0G1H103JT0Y0N" (id 1) (at 135.89 120.65 90)
+      (effects (font (size 1.27 1.27)) (justify left))
+    )
