File: Piezo_Drive.kicad_sch (KiCad schematic)
At the start: 72 parts, among them J26 AudioJack3, Q1 MMBT3906, Q2 mmbt3904, Q3 2SCR573, Q4 2SAR573, Q5 MMBT3906, Q6 mmbt3904, Q7 2SCR573, Q8 2SAR573, U7 ADA4075-2

Commit message: Preliminary layout of analog portions
Parts:
- removed J26: AudioJack3, Connector_Audio:Jack_3.5mm_CUI_SJ-3524-SMT_Horizontal, symbol Connector:AudioJack3
- added J26: SJ1-3514-SMT-TR, SJ13514SMTTR, symbol SamacSys_Parts:SJ1-3514-SMT-TR
- added J32: SMA, Connector_Coaxial:SMA_Amphenol_132134-10_Vertical, symbol Connector:Conn_Coaxial
Connections:
- net GND: now also J26.1 (SLEEVE)
- net bias_l: no longer C67.1, D7.2 (A), R92.2
- net piezo_slow: now reaches C147.1, C158.1, R138.2
- net piezo_slow: now also J26.2 (TIP), J32.2 (Ext)
- net piezo_fast: now reaches R162.2
- net piezo_fast: now also J26.3 (RING), J32.1 (In)
- new net: C67.1, D7.2 (A), R92.2
- no-connect marks 0 -> 2
Other:
- note added: "PJ-240-SMT PJ-342B-TX-SMT"
- moved on the sheet: C139, C140, C141, C142, C143, C144, C147, C158, C159, C66, C67, C68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

Commit message: Analog section complete!
Parts:
- removed C158: OVK151M1VTR-1013, Capacitor_SMD:CP_Elec_10x10.5, symbol Device:CP
- removed R97: 100, Resistor_SMD:R_0805_2012Metric, symbol Device:R
- added C158, C160: 0.1uF, Capacitor_SMD:C_0603_1608Metric_Pad1.08x0.95mm_HandSolder, symbol Device:C
- added C161: OVK151M1VTR-1013, Capacitor_SMD:CP_Elec_10x10.5, symbol Device:CP
- added IC2: TMUX7219DGKRQ1, SOP65P490X110-8N, symbol SamacSys_Parts:TMUX7219DGKRQ1
- added J33: Conn_01x04, Connector_PinHeader_2.54mm:PinHeader_1x04_P2.54mm_Vertical, symbol Connector_Generic:Conn_01x04
- added R166: 270, Resistor_SMD:R_0805_2012Metric, symbol Device:R
- added TP5: tp, TestPoint:TestPoint_Pad_D1.0mm, symbol Connector:TestPoint
- R14: value 270 -> 150
- R95: value 270 -> 100
- R99: value 100 -> 150
Connections:
- net +28V: now also C158.1, IC2.4 (VDD)
- net -5VA: now also C160.1, IC2.7 (VSS)
- net GND: now also C158.2, C160.2, C161.2, IC2.3 (GND), J33.1 (Pin_1), J33.4 (Pin_4)
- net bias_l: now also C67.1, D7.2 (A), R92.2
- net piezo_slow: now also R138.1, IC2.1 (D), R166.2; no longer R138.2
- net at R105.2, R106.1: now also R138.2; no longer R138.1
- net input renamed fast_in_A
- net fast_in_A: no longer R95.1
- net offset renamed fast_in_B
- new net: IC2.2 (S1), TP5.1
- new net: C161.1, IC2.8 (S2), R166.1
- new net CSwitch_EN: IC2.5 (EN), J33.2 (Pin_2)
- new net CSwitch_SEL: IC2.6 (SEL), J33.3 (Pin_3)
- new net slow_in: R95.1
Other:
- note added: "better op amp OPA2992 LME49860 ADA4522-2 LT1124 LT1037/LT1137 LT1128"
- moved on the sheet: C139, C141, C142, C145, C146, C147, C159, C68, C69, C70, C71, C72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

Commit message: First finished draft
Parts:
- added R181: 3k3, Resistor_SMD:R_1206_3216Metric, symbol Device:R
- C161: symbol Device:CP -> Device:C_Polarized
- IC2: footprint SOP65P490X110-8N -> SamacSys_Parts:SOP65P490X110-8N
- J26: footprint SJ13514SMTTR -> SamacSys_Parts:SJ13514SMTTR
- U7: footprint (none) -> Package_SO:SOIC-8_3.9x4.9mm_P1.27mm
Connections:
- net out_B_o: now reaches R160.2, R161.1, R162.1
- net out_B_o: now also R181.2
- net at C139.2, C140.1, R101.1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: now also R181.1
Other:
- moved on the sheet: C140, R163, R164
Changed lines of the file:
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@@
   (junction (at 243.84 55.88) (diameter 0) (color 0 0 0 0)
+  )
+  (junction (at 222.25 92.71) (diameter 0) (color 0 0 0 0)
   )
   (junction (at 139.7 171.45) (diameter 0) (color 0 0 0 0)
@@
     (stroke (width 0) (type default) (color 0 0 0 0))
   )
+  (wire (pts (xy 222.25 92.71) (xy 226.06 92.71))
+    (stroke (width 0) (type default) (color 0 0 0 0))
+  )
   (wire (pts (xy 213.36 115.57) (xy 213.36 123.19))
     (stroke (width 0) (type default) (color 0 0 0 0))
   )
-  (wire (pts (xy 72.39 106.68) (xy 72.39 114.3))
+  (wire (pts (xy 72.39 106.68) (xy 72.39 115.57))
     (stroke (width 0) (type default) (color 0 0 0 0))
   )
@@
     (stroke (width 0) (type default) (color 0 0 0 0))
   )
-  (wire (pts (xy 229.87 92.71) (xy 234.95 92.71))
+  (wire (pts (xy 233.68 92.71) (xy 234.95 92.71))
     (stroke (width 0) (type default) (color 0 0 0 0))
   )
@@
     (stroke (width 0) (type default) (color 0 0 0 0))
   )
-  (wire (pts (xy 82.55 121.92) (xy 82.55 127))
+  (wire (pts (xy 82.55 123.19) (xy 82.55 132.08))
     (stroke (width 0) (type default) (color 0 0 0 0))
   )
@@
     (stroke (width 0) (type default) (color 0 0 0 0))
   )
+  (wire (pts (xy 222.25 105.41) (xy 222.25 123.19))
+    (stroke (width 0) (type default) (color 0 0 0 0))
+  )
   (wire (pts (xy 229.87 45.72) (xy 232.41 45.72))
     (stroke (width 0) (type default) (color 0 0 0 0))
@@
     (stroke (width 0) (type default) (color 0 0 0 0))
   )
-  (wire (pts (xy 72.39 121.92) (xy 72.39 127))
-    (stroke (width 0) (type default) (color 0 0 0 0))
-  )
-  (wire (pts (xy 82.55 106.68) (xy 82.55 114.3))
+  (wire (pts (xy 72.39 123.19) (xy 72.39 132.08))
+    (stroke (width 0) (type default) (color 0 0 0 0))
+  )
+  (wire (pts (xy 82.55 106.68) (xy 82.55 115.57))
     (stroke (width 0) (type default) (color 0 0 0 0))
   )
@@
   )
   (wire (pts (xy 83.82 62.23) (xy 83.82 69.85))
+    (stroke (width 0) (type default) (color 0 0 0 0))
+  )
+  (wire (pts (xy 222.25 97.79) (xy 222.25 92.71))
     (stroke (width 0) (type default) (color 0 0 0 0))
   )
@@
     (effects (font (size 1.27 1.27)) (justify right bottom))
   )
-  (label "out_A_p" (at 82.55 127 270)
+  (label "out_A_p" (at 82.55 132.08 270)
     (effects (font (size 1.27 1.27)) (justify right bottom))
   )
-  (label "out_A_n" (at 72.39 127 270)
+  (label "out_A_n" (at 72.39 132.08 270)
+    (effects (font (size 1.27 1.27)) (justify right bottom))
+  )
+  (label "out_B_o" (at 222.25 123.19 270)
     (effects (font (size 1.27 1.27)) (justify right bottom))
   )
@@
   (label "out_A_n" (at 129.54 97.79 0)
     (effects (font (size 1.27 1.27)) (justify left bottom))
+  )
+  (label "out_B_o" (at 261.62 78.74 180)
+    (effects (font (size 1.27 1.27)) (justify right bottom))
   )
   (label "out_A_p" (at 129.54 63.5 0)
@@
       (effects (font (size 1.27 1.27)) (justify left))
     )
-    (property "Footprint" "" (id 2) (at 132.08 168.91 0)
+    (property "Footprint" "Package_SO:SOIC-8_3.9x4.9mm_P1.27mm" (id 2) (at 132.08 168.91 0)
       (effects (font (size 1.27 1.27)) hide)
     )
@@
       (effects (font (size 1.27 1.27)) (justify right))
     )
-    (property "Footprint" "SOP65P490X110-8N" (id 2) (at 165.1 111.76 0)
+    (property "Footprint" "SamacSys_Parts:SOP65P490X110-8N" (id 2) (at 165.1 111.76 0)
       (effects (font (size 1.27 1.27)) (justify left) hide)
     )
@@
     (pin "8")
   )
-  (symbol (lib_id "Device:CP") (at 170.18 128.27 90) (unit 1)
+  (symbol (lib_id "Device:C_Polarized") (at 170.18 128.27 90) (unit 1)
     (in_bom yes) (on_board yes)
     (property "Reference" "C161" (id 0) (at 167.64 127 0)
@@
     (pin "2")
   )
+  (symbol (lib_id "Device:R") (at 222.25 101.6 0) (unit 1)
+    (in_bom yes) (on_board yes)
+    (property "Reference" "R181" (id 0) (at 224.79 100.3299 0)
+      (effects (font (size 1.27 1.27)) (justify left))
+    )
+    (property "Value" "3k3" (id 1) (at 224.79 106.68 90)
+      (effects (font (size 1.27 1.27)) (justify left))
+    )
+    (property "Footprint" "Resistor_SMD:R_1206_3216Metric" (id 2) (at 220.472 101.6 90)
+      (effects (font (size 1.27 1.27)) hide)
+    )
+    (property "Datasheet" "~" (id 3) (at 222.25 101.6 0)
+      (effects (font (size 1.27 1.27)) hide)
+    )
+    (pin "1")
+    (pin "2")
+  )
   (symbol (lib_id "power:GND") (at 195.58 109.22 0) (mirror y) (unit 1)
     (in_bom yes) (on_board yes)
@@
     (pin "1")
   )
-  (symbol (lib_id "Device:R") (at 72.39 118.11 0) (unit 1)
-    (in_bom yes) (on_board yes)
-    (property "Reference" "R163" (id 0) (at 74.93 116.8399 0)
-      (effects (font (size 1.27 1.27)) (justify left))
-    )
-    (property "Value" "2k2" (id 1) (at 74.93 123.19 90)
-      (effects (font (size 1.27 1.27)) (justify left))
-    )
-    (property "Footprint" "Resistor_SMD:R_1206_3216Metric" (id 2) (at 70.612 118.11 90)
-      (effects (font (size 1.27 1.27)) hide)
-    )
-    (property "Datasheet" "~" (id 3) (at 72.39 118.11 0)
+  (symbol (lib_id "Device:R") (at 72.39 119.38 0) (unit 1)
+    (in_bom yes) (on_board yes)
+    (property "Reference" "R163" (id 0) (at 74.93 118.1099 0)
+      (effects (font (size 1.27 1.27)) (justify left))
+    )
+    (property "Value" "2k2" (id 1) (at 74.93 124.46 90)
+      (effects (font (size 1.27 1.27)) (justify left))
+    )
+    (property "Footprint" "Resistor_SMD:R_1206_3216Metric" (id 2) (at 70.612 119.38 90)
+      (effects (font (size 1.27 1.27)) hide)
+    )
+    (property "Datasheet" "~" (id 3) (at 72.39 119.38 0)
       (effects (font (size 1.27 1.27)) hide)
     )
@@
     (property "Reference" "J26" (id 0) (at 69.85 168.91 0))
     (property "Value" "SJ1-3514-SMT-TR" (id 1) (at 69.85 171.45 0))
-    (property "Footprint" "SJ13514SMTTR" (id 2) (at 86.36 173.99 0)
+    (property "Footprint" "SamacSys_Parts:SJ13514SMTTR" (id 2) (at 86.36 173.99 0)
       (effects (font (size 1.27 1.27)) (justify left) hide)
     )
@@
     (pin "3")
   )
-  (symbol (lib_id "Device:R") (at 82.55 118.11 0) (unit 1)
-    (in_bom yes) (on_board yes)
-    (property "Reference" "R164" (id 0) (at 85.09 116.8399 0)
-      (effects (font (size 1.27 1.27)) (justify left))
-    )
-    (property "Value" "2k2" (id 1) (at 85.09 123.19 90)
-      (effects (font (size 1.27 1.27)) (justify left))
-    )
-    (property "Footprint" "Resistor_SMD:R_1206_3216Metric" (id 2) (at 80.772 118.11 90)
-      (effects (font (size 1.27 1.27)) hide)
-    )
-    (property "Datasheet" "~" (id 3) (at 82.55 118.11 0)
+  (symbol (lib_id "Device:R") (at 82.55 119.38 0) (unit 1)
+    (in_bom yes) (on_board yes)
+    (property "Reference" "R164" (id 0) (at 85.09 118.1099 0)
+      (effects (font (size 1.27 1.27)) (justify left))
+    )
+    (property "Value" "2k2" (id 1) (at 85.09 124.46 90)
+      (effects (font (size 1.27 1.27)) (justify left))
+    )
+    (property "Footprint" "Resistor_SMD:R_1206_3216Metric" (id 2) (at 80.772 119.38 90)
+      (effects (font (size 1.27 1.27)) hide)
+    )
+    (property "Datasheet" "~" (id 3) (at 82.55 119.38 0)
       (effects (font (size 1.27 1.27)) hide)
     )
@@
     (pin "1")
   )
-  (symbol (lib_id "Device:C") (at 226.06 92.71 90) (unit 1)
-    (in_bom yes) (on_board yes)
-    (property "Reference" "C140" (id 0) (at 226.06 85.09 90))
-    (property "Value" "22p" (id 1) (at 226.06 87.63 90))
-    (property "Footprint" "Capacitor_SMD:C_0603_1608Metric" (id 2) (at 229.87 91.7448 0)
-      (effects (font (size 1.27 1.27)) hide)
-    )
-    (property "Datasheet" "~" (id 3) (at 226.06 92.71 0)
-      (effects (font (size 1.27 1.27)) hide)
-    )
+  (symbol (lib_id "Device:C") (at 229.87 92.71 90) (unit 1)
+    (in_bom yes) (on_board yes)
+    (property "Reference" "C140" (id 0) (at 229.87 85.09 90))
+    (property "Value" "22p" (id 1) (at 229.87 87.63 90))
+    (property "Footprint" "Capacitor_SMD:C_0603_1608Metric" (id 2) (at 233.68 91.7448 0)
+      (effects (font (size 1.27 1.27)) hide)
+    )
+    (property "Datasheet" "~" (id 3) (at 229.87 92.71 0)
+      (effects (font (size 1.27 1.27)) hide)
+    )
