File: ch32v307_core.kicad_sch (KiCad schematic)
At the start: 64 parts, among them J1 U254-051T-4BH83-S1S, J10 Conn_01x12_Male, J2 U254-051T-4BH83-S1S, J5 debug, J6 Clock_in, J7 Conn_01x08, J8 Conn_01x30_Male, J9 Conn_01x21_Male, U1 CH32V307RCT6, Y1 X32258MOB4SI

Commit message: Digital section half finished
Parts:
- removed J10: Conn_01x12_Male, Connector_PinHeader_2.54mm:PinHeader_1x12_P2.54mm_Vertical, symbol Connector:Conn_01x12_Male
- removed J8: Conn_01x30_Male, Connector_PinHeader_2.54mm:PinHeader_1x27_P2.54mm_Vertical, symbol Connector:Conn_01x27_Male
- removed J9: Conn_01x21_Male, Connector_PinHeader_2.54mm:PinHeader_1x21_P2.54mm_Vertical, symbol Connector:Conn_01x21_Male
- removed R2, R3: 27, Resistor_SMD:R_0603_1608Metric_Pad0.98x0.95mm_HandSolder, symbol Device:R
- added J10: B-2100N06P-B111, Connector_PinHeader_2.54mm:PinHeader_2x03_P2.54mm_Vertical_SMD, symbol Connector_Generic:Conn_02x03_Odd_Even
- added J36: MMCX, SamacSys_Parts:MMCX_Molex_SMT_734152061_Vertical, symbol Connector:Conn_Coaxial
- added J37, J38: Conn_01x16, Connector_PinHeader_2.54mm:PinHeader_1x16_P2.54mm_Vertical, symbol Connector_Generic:Conn_01x16
- added J8: Conn_01x08, Connector_PinHeader_2.54mm:PinHeader_1x08_P2.54mm_Vertical, symbol Connector_Generic:Conn_01x08
- added J9: U.FL, Connector_Coaxial:U.FL_Hirose_U.FL-R-SMT-1_Vertical, symbol Connector:Conn_Coaxial
- added R169, R170, R171, R172, R173, R174: 27, Resistor_SMD:R_0603_1608Metric_Pad0.98x0.95mm_HandSolder, symbol Device:R
- added R175: 4k7, Resistor_SMD:R_0603_1608Metric_Pad0.98x0.95mm_HandSolder, symbol Device:R
- J7: footprint Connector_PinHeader_1.27mm:PinHeader_1x08_P1.27mm_Vertical -> Connector_PinHeader_2.54mm:PinHeader_1x08_P2.54mm_Vertical
- R17: value 4k7 -> 27
Connections:
- net GND: now also J10.1 (Pin_1), J10.6 (Pin_6), J36.2 (Ext), J37.11 (Pin_11), J37.16 (Pin_16), J37.2 (Pin_2), J37.4 (Pin_4), J37.7 (Pin_7), J38.12 (Pin_12), J38.16 (Pin_16), J38.4 (Pin_4), J38.8 (Pin_8), J8.1 (Pin_1), J8.8 (Pin_8), J9.2 (Ext)
- net PB0: now also R29.1; no longer R30.1
- net PB1: now also R30.1; no longer R29.1
- net PB10_I2C2_SCL: now also R27.1; no longer R19.1, R28.1
- net PB11_I2C2_SDA: now also R28.1; no longer R18.1, R27.1
- net PB8_I2C1_SCL: now also R17.1; no longer R16.1
- net PB9_I2C1_SDA: now also R174.1; no longer R17.1
- net PC0: now also R172.1
- net PC1: now also R173.1
- net PC13_TPR_RTC: now also J8.5 (Pin_5)
- net PC14_OSC32_I: now also J8.6 (Pin_6)
- net PC15_OSC32_O: now also J8.7 (Pin_7)
- net PC2: now also R171.1
- net PC4: now also R170.1
- net PC5: now also R169.1
- net at R40.2: now also J38.15 (Pin_15)
- net at R41.2: now also J38.14 (Pin_14)
- net at R39.2: now also J36.1 (In), J37.3 (Pin_3)
- net at R10.2: now also J38.11 (Pin_11)
- net at R26.2: now also J37.15 (Pin_15)
- net at R8.2: now also J38.7 (Pin_7)
- net at R5.2: now also J10.5 (Pin_5)
- net at R7.2: now also J10.2 (Pin_2)
- net at R9.2: now also J38.10 (Pin_10)
- net at R28.2: now also R18.2, J37.13 (Pin_13)
- net at R27.2: now also R19.2, J37.12 (Pin_12)
- net at R4.2: now also J10.3 (Pin_3)
- net at R6.2: now also J10.4 (Pin_4)
- net at R29.2: now also J37.9 (Pin_9)
- net at R30.2: now also J37.10 (Pin_10)
- net +3V3 renamed +3.3V
- net +3.3V: now also R16.1, R18.1, R19.1, J37.1 (Pin_1), J37.14 (Pin_14), J37.8 (Pin_8), J38.1 (Pin_1), J38.13 (Pin_13), J38.5 (Pin_5), J38.9 (Pin_9), J8.4 (Pin_4), R175.1; no longer R16.2, R17.2, R18.2, R19.2
- new net: J38.3 (Pin_3), R173.2
- new net: J8.2 (Pin_2), R16.2, R17.2
- new net: J38.6 (Pin_6), R171.2
- new net: J37.6 (Pin_6), R169.2
- new net: J38.2 (Pin_2), R172.2
- new net: J37.5 (Pin_5), R170.2
- new net: J8.3 (Pin_3), R174.2, R175.2
Other:
- moved on the sheet: C1, C2, C29, C3, C37, C38, C39, C4, C5, C6, J5, J6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

Commit message: First finished draft
Parts:
- removed J5: debug, Connector_PinHeader_2.54mm:PinHeader_1x06_P2.54mm_Vertical, symbol Connector:Conn_01x06_Male
- added C171: X7R 0.1u, Capacitor_SMD:C_0603_1608Metric_Pad1.08x0.95mm_HandSolder, symbol Device:C
- added J39, J40: B-2100N06P-B111, Connector_PinHeader_2.54mm:PinHeader_2x03_P2.54mm_Vertical_SMD, symbol Connector_Generic:Conn_02x03_Odd_Even
- added JA0, JA1, JC0, JC1: MMCX, SamacSys_Parts:MMCX_Molex_SMT_734152061_Vertical, symbol Connector:Conn_Coaxial
- added JA2, JA3, JC2, JC3, JC5: U.FL, Connector_Coaxial:U.FL_Hirose_U.FL-R-SMT-1_Vertical, symbol Connector:Conn_Coaxial
- added JP18: sjp, Jumper:SolderJumper-3_P1.3mm_Open_RoundedPad1.0x1.5mm, symbol Jumper:SolderJumper_3_Open
- renumbered J36 to JA4, J9 to JC4
Connections:
- net +3.3V: now also J40.1 (Pin_1), JP18.3 (B); no longer U1.13 (VDDA)
- net GND: now also C171.1, J39.1 (Pin_1), J39.2 (Pin_2), J39.6 (Pin_6), J40.6 (Pin_6), JA0.2 (Ext), JA1.2 (Ext), JA2.2 (Ext), JA3.2 (Ext), JC0.2 (Ext), JC1.2 (Ext), JC2.2 (Ext), JC3.2 (Ext), JC5.2 (Ext)
- net PA0: now also JA0.1 (In)
- net PA1: now also JA1.1 (In)
- net PC2: now also JC2.1 (In)
- net PC3: now also JC3.1 (In)
- net PC4: now also JC4.1 (In)
- net PC5: now also JC5.1 (In)
- net SPI3_CS: now also R6.1; no longer R4.1
- net SPI3_MISO: now also R4.1; no longer R6.1
- net SWCLK: now also J40.2 (Pin_2)
- net SWDIO: now also J40.4 (Pin_4)
- net PC1_R: now reaches J38.3 (Pin_3), R173.2
- net PC1_R: now also JC1.1 (In)
- net at R34.2: now also J39.3 (Pin_3)
- net PC0_R: now reaches J38.2 (Pin_2), R172.2
- net PC0_R: now also JC0.1 (In)
- net PA2_R: now reaches J38.14 (Pin_14), R41.2
- net PA2_R: now also JA2.1 (In)
- net at R35.2: now also J39.5 (Pin_5)
- net PA3_R: now reaches J38.15 (Pin_15), R40.2
- net PA3_R: now also JA3.1 (In)
- net at R33.2: now also J39.4 (Pin_4)
- net at R31.2: now also J40.3 (Pin_3)
- net at R32.2: now also J40.5 (Pin_5)
- net Vin renamed VUSB
- new net: C171.2, JP18.2 (C), U1.13 (VDDA)
- new net +3.3VA: JP18.1 (A)
- no-connect marks 0 -> 2
Other:
- moved on the sheet: J10, J38, J7, JC4, R10, R171, R172, R173, R31, R32, R33, R34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

Commit message: Version 1.0 submitted to JLCPCB
Parts:
- C171, C2, C29, C37, C38, C39, C6: value X7R 0.1u -> 0.1u
- D1, D2: value B5819W -> B5819W SL
- J6: value Clock_in -> DNP U.FL
- JA0, JA1, JA4, JC0, JC1: value MMCX -> DNP MMCX
- JA2, JA3, JC2, JC3, JC4, JC5: value U.FL -> DNP U.FL
- renumbered S_BOOT1 to S_BOOT0
Connections:
- net +3.3V: now also J39.2 (Pin_2)
- net GND: no longer J39.2 (Pin_2)
Other:
- moved on the sheet: J7
