File: power_3.kicad_sch (KiCad schematic)
At the start: 0 parts

Commit message: First finished draft
Parts:
- added C162, C165: tant 10u, Capacitor_Tantalum_SMD:CP_EIA-3216-18_Kemet-A, symbol Device:C_Polarized
- added C163, C169: 4.7uF, Capacitor_SMD:C_1206_3216Metric_Pad1.33x1.80mm_HandSolder, symbol Device:C
- added C164: 0.1uF, Capacitor_SMD:C_0805_2012Metric_Pad1.18x1.45mm_HandSolder, symbol Device:C
- added C166, C25: x7r 1u, Capacitor_SMD:C_0805_2012Metric, symbol Device:C
- added C167: 10n, Capacitor_SMD:C_0805_2012Metric_Pad1.18x1.45mm_HandSolder, symbol Device:C
- added C168: dnp, Capacitor_SMD:C_1206_3216Metric_Pad1.33x1.80mm_HandSolder, symbol Device:C
- added C170: tant cap, Capacitor_Tantalum_SMD:CP_EIA-3528-15_AVX-H_Pad1.50x2.35mm_HandSolder, symbol Device:C_Polarized
- added D17: B5819W SL, Diode_SMD:D_SOD-123F, symbol Device:D
- added IC3: ADP7118AUJZ-3.3-R7, SamacSys_Parts:SOT95P280X100-5N, symbol SamacSys_Parts:ADP7118AUJZ-2.5-R7
- added J5: Conn_Coaxial, Connector_Coaxial:U.FL_Hirose_U.FL-R-SMT-1_Vertical, symbol Connector:Conn_Coaxial
- added R176, R2: dnp, Resistor_SMD:R_0805_2012Metric_Pad1.20x1.40mm_HandSolder, symbol Device:R
- added R3: 0, Resistor_SMD:R_0805_2012Metric_Pad1.20x1.40mm_HandSolder, symbol Device:R
- added U27: AMS1117-3.3, Package_TO_SOT_SMD:SOT-223-3_TabPin2, symbol Regulator_Linear:AMS1117-3.3
Connections:
- new net: C167.2, C168.2, R2.1
- new net +3.3V: C165.1, C166.1, U27.2 (VO)
- new net +3.3VA: C167.1, C168.1, C169.1, C170.1, D17.1 (K), IC3.5 (VOUT), J5.1 (In), R3.1
- new net +5VA: C163.1, C164.1, IC3.1 (VIN), IC3.3 (EN)
- new net GND: C162.2, C163.2, C164.2, C165.2, C166.2, C169.2, C170.2, C25.2, D17.2 (A), IC3.2 (GND), J5.2 (Ext), R176.2, U27.1 (GND)
- new net VUSB: C162.1, C25.1, U27.3 (VI)
- new net sense_vdd: IC3.4 (SENSE/ADJ), R176.1, R2.2, R3.2

Commit message: Moved 3.3VA supply out of the ADC area, to have that area cleaner
Parts:
- R176, R2, R3: footprint Resistor_SMD:R_0805_2012Metric_Pad1.20x1.40mm_HandSolder -> Resistor_SMD:R_0805_2012Metric
Changed lines of the file:
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@@
       (effects (font (size 1.27 1.27)) (justify right))
     )
-    (property "Footprint" "Resistor_SMD:R_0805_2012Metric_Pad1.20x1.40mm_HandSolder" (id 2) (at 189.103 64.77 90)
+    (property "Footprint" "Resistor_SMD:R_0805_2012Metric" (id 2) (at 189.103 64.77 90)
       (effects (font (size 1.27 1.27)) hide)
     )
@@
       (effects (font (size 1.27 1.27)) (justify right))
     )
-    (property "Footprint" "Resistor_SMD:R_0805_2012Metric_Pad1.20x1.40mm_HandSolder" (id 2) (at 182.245 71.882 90)
+    (property "Footprint" "Resistor_SMD:R_0805_2012Metric" (id 2) (at 182.245 71.882 90)
       (effects (font (size 1.27 1.27)) hide)
     )
@@
       (effects (font (size 1.27 1.27)) (justify right))
     )
-    (property "Footprint" "Resistor_SMD:R_0805_2012Metric_Pad1.20x1.40mm_HandSolder" (id 2) (at 189.103 81.28 90)
-      (effects (font (size 1.27 1.27)) hide)
-    )
+    (property "Footprint" "Resistor_SMD:R_0805_2012Metric" (id 2) (at 189.103 81.28 90)
+      (effects (font (size 1.27 1.27)) hide)
+    )

Commit message: Version 1.0 submitted to JLCPCB
Parts:
- C162, C165: value tant 10u -> TAJA106K016RNJ
- C166, C25: value x7r 1u -> 1uF
- C167: value 10n -> CGA4C2C0G1H103JT0Y0N
- D17: footprint Diode_SMD:D_SOD-123F -> Diode_SMD:D_SOD-123
- J5: value Conn_Coaxial -> DNP U.FL
- R3: value 0 -> 0R
Changed lines of the file:
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@@
       (effects (font (size 1.27 1.27)) (justify right))
     )
-    (property "Value" "0" (id 1) (at 189.103 65.913 0)
+    (property "Value" "0R" (id 1) (at 189.103 65.913 0)
       (effects (font (size 1.27 1.27)) (justify right))
     )
@@
     (in_bom yes) (on_board yes)
     (property "Reference" "J5" (id 0) (at 231.2162 51.1048 0))
-    (property "Value" "Conn_Coaxial" (id 1) (at 231.2162 53.4162 0))
+    (property "Value" "DNP U.FL" (id 1) (at 231.2162 53.4162 0))
     (property "Footprint" "Connector_Coaxial:U.FL_Hirose_U.FL-R-SMT-1_Vertical" (id 2) (at 233.045 57.15 0)
       (effects (font (size 1.27 1.27)) hide)
@@
       (effects (font (size 1.27 1.27)) (justify left))
     )
-    (property "Value" "10n" (id 1) (at 168.91 60.96 0)
+    (property "Value" "CGA4C2C0G1H103JT0Y0N" (id 1) (at 168.91 60.96 0)
       (effects (font (size 1.27 1.27)) (justify left))
     )
@@
   )
   (symbol (lib_id "Device:C_Polarized") (at 82.55 137.16 0) (unit 1)
-    (in_bom yes) (on_board yes) (fields_autoplaced)
+    (in_bom yes) (on_board yes)
     (property "Reference" "C162" (id 0) (at 86.36 135.0009 0)
       (effects (font (size 1.27 1.27)) (justify left))
     )
-    (property "Value" "tant 10u" (id 1) (at 86.36 137.5409 0)
+    (property "Value" "TAJA106K016RNJ" (id 1) (at 73.66 146.05 0)
       (effects (font (size 1.27 1.27)) (justify left))
     )
@@
       (effects (font (size 1.27 1.27)) (justify left))
     )
-    (property "Value" "x7r 1u" (id 1) (at 71.12 138.4299 0)
+    (property "Value" "1uF" (id 1) (at 71.12 138.4299 0)
       (effects (font (size 1.27 1.27)) (justify left))
     )
@@
       (effects (font (size 1.27 1.27)) (justify left))
     )
-    (property "Footprint" "Diode_SMD:D_SOD-123F" (id 2) (at 202.565 69.85 0)
+    (property "Footprint" "Diode_SMD:D_SOD-123" (id 2) (at 202.565 69.85 0)
       (effects (font (size 1.27 1.27)) hide)
     )
@@
       (effects (font (size 1.27 1.27)) (justify left))
     )
-    (property "Value" "x7r 1u" (id 1) (at 134.62 138.4299 0)
+    (property "Value" "1uF" (id 1) (at 134.62 138.4299 0)
       (effects (font (size 1.27 1.27)) (justify left))
     )
@@
   )
   (symbol (lib_id "Device:C_Polarized") (at 114.3 137.16 0) (unit 1)
-    (in_bom yes) (on_board yes) (fields_autoplaced)
+    (in_bom yes) (on_board yes)
     (property "Reference" "C165" (id 0) (at 118.11 135.0009 0)
       (effects (font (size 1.27 1.27)) (justify left))
     )
-    (property "Value" "tant 10u" (id 1) (at 118.11 137.5409 0)
-      (effects (font (size 1.27 1.27)) (justify left))
-    )
+    (property "Value" "TAJA106K016RNJ" (id 1) (at 107.95 146.05 0)
+      (effects (font (size 1.27 1.27)) (justify left))
+    )
