File: reference_and_buffer.kicad_sch (KiCad schematic)
At the start: 37 parts, among them IC9 LTC6655BHMS8-4.096#PBF, U11 OPA388, U12 ADR421ARZ, U13 THS4281, U22 OPA388

Commit message: First finished draft
Parts:
- C115: symbol Device:CP -> Device:C_Polarized
Changed lines of the file:
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@@
     (pin "2")
   )
-  (symbol (lib_id "Device:CP") (at 116.84 158.75 0) (mirror y) (unit 1)
+  (symbol (lib_id "Device:C_Polarized") (at 116.84 158.75 0) (mirror y) (unit 1)
     (in_bom yes) (on_board yes)
     (property "Reference" "C115" (id 0) (at 118.11 166.37 0)

Commit message: Version 1.0 submitted to JLCPCB
Parts:
- R137: value 0 -> 0R
Changed lines of the file:
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@@
       (effects (font (size 1.27 1.27)) (justify right))
     )
-    (property "Value" "0" (id 1) (at 119.38 149.8599 0)
+    (property "Value" "0R" (id 1) (at 119.38 149.8599 0)
       (effects (font (size 1.27 1.27)) (justify right))
     )
